File: display driver shift reg.sch (EAGLE design)
At the start: 175 parts, among them IC1 74HC166, IC10 74HC138, IC11 74HC595, IC12 74HC595, IC13 74HC595, IC14 74HC595, IC15 74HC595, IC16 74HC595, IC17 74HC595, IC18 74HC595, IC19 74HC595, IC2 74HC688, IC20 74HC595, IC21 74HC595, IC22 74HC595, IC23 74HC595, IC24 74HC595, IC25 74HC595, IC26 74HC595, IC27 74HC595, IC28 74HC08, IC29 74LS245N, IC3 74HC32, IC30 74LS245N, IC31 74LS245N, IC4 74HC74, IC5 74HC08, IC6 74HC393, IC7 74HC04, IC8 74HC688, IC9 74HC573

Commit message: Update bus pins, add power and decoupling
Parts:
- removed IC30, IC31: 74LS245N, 74xx-us:74LS245N
- added C10, C11, C12, C13, C14, C15, C16, C17, C18, C19, C20, C21, C22, C23, C24, C25, C26, C27, C28, C29, C3, C30, C31, C32, C33, C4, C5, C6, C7, C8, C9: 100nF, rcl:C-EU050-025X075
- added U2, U3: 74LS245N, 74xx-us:74LS245N
- renumbered IC1 to U11, IC10 to U14, IC11 to U15, IC12 to U16, IC13 to U17, IC14 to U18, IC15 to U19, IC16 to U20, IC17 to U21, IC18 to U22, IC19 to U23, IC2 to U4, IC20 to U24, IC21 to U25, IC22 to U26, IC23 to U27, IC24 to U28, IC25 to U29, IC26 to U30, IC27 to U31, IC28 to U12, IC29 to U1, IC3 to U10, IC4 to U7, IC5 to U8, IC6 to U9, IC7 to U6, IC8 to U5, IC9 to U13, SV5 to BUS
Connections:
- net !INT!: now also BUS-11.S; no longer BUS-31.S
- net !IORQ!: now also U3A.B3; no longer IC31A.B3
- net !NMI!: now also BUS-12.S; no longer BUS-32.S
- net !RESET!: now also U3A.B7; no longer IC31A.B7
- net !WAIT!: now also BUS-10.S; no longer BUS-30.S
- net !WR!: now also U3A.B5; no longer IC31A.B5
- net +5V: now also BUS-3.S, C10.1, C11.1, C12.1, C13.1, C14.1, C15.1, C16.1, C17.1, C18.1, C19.1, C20.1, C21.1, C22.1, C23.1, C24.1, C25.1, C26.1, C27.1, C28.1, C29.1, C3.1, C30.1, C31.1, C32.1, C33.1, C4.1, C5.1, C6.1, C7.1, C8.1, C9.1, U10P.VCC, U11P.VCC, U12P.VCC, U13P.VCC, U14P.VCC, U15P.VCC, U16P.VCC, U17P.VCC, U18P.VCC, U19P.VCC, U1P.VCC, U20P.VCC, U21P.VCC, U22P.VCC, U23P.VCC, U24P.VCC, U25P.VCC, U26P.VCC, U27P.VCC, U28P.VCC, U29P.VCC, U2A.DIR, U2P.VCC, U30P.VCC, U31P.VCC, U3A.DIR, U3P.VCC, U4P.VCC, U5P.VCC, U6P.VCC, U7P.VCC, U8P.VCC, U9P.VCC; no longer BUS-2.S, IC30A.DIR, IC31A.DIR
- net A0: now also U2A.B1; no longer IC30A.B1
- net A1: now also U2A.B2; no longer IC30A.B2
- net A2: now also U2A.B3; no longer IC30A.B3
- net A3: now also U2A.B4; no longer IC30A.B4
- net A4: now also U2A.B5; no longer IC30A.B5
- net A5: now also U2A.B6; no longer IC30A.B6
- net A6: now also U2A.B7; no longer IC30A.B7
- net A7: now also U2A.B8; no longer IC30A.B8
- net CLK: now also U3A.B8; no longer IC31A.B8
- net GND: now also BUS-2.S, BUS-31.S, BUS-32.S, C10.2, C11.2, C12.2, C13.2, C14.2, C15.2, C16.2, C17.2, C18.2, C19.2, C20.2, C21.2, C22.2, C23.2, C24.2, C25.2, C26.2, C27.2, C28.2, C29.2, C3.2, C30.2, C31.2, C32.2, C33.2, C4.2, C5.2, C6.2, C7.2, C8.2, C9.2, U10P.GND, U11P.GND, U12P.GND, U13P.GND, U14P.GND, U15P.GND, U16P.GND, U17P.GND, U18P.GND, U19P.GND, U1P.GND, U20P.GND, U21P.GND, U22P.GND, U23P.GND, U24P.GND, U25P.GND, U26P.GND, U27P.GND, U28P.GND, U29P.GND, U2A.G, U2P.GND, U30P.GND, U31P.GND, U3A.A6, U3A.G, U3P.GND, U4P.GND, U5P.GND, U6P.GND, U7P.GND, U8P.GND, U9P.GND; no longer BUS-13.S, BUS-14.S, BUS-23.S, BUS-24.S, BUS-3.S, IC30A.G, IC31A.A6, IC31A.G
- net N$19: now also BUS-33.S, U2A.A1; no longer BUS-5.S, U1A.A1
- net N$20: now also BUS-34.S, U2A.A2; no longer BUS-6.S, U1A.A2
- net N$22: now also BUS-35.S, U2A.A3; no longer BUS-7.S, U1A.A3
- net N$23: now also BUS-36.S, U2A.A4; no longer BUS-8.S, U1A.A4
- net N$26: now also BUS-37.S, U2A.A5; no longer BUS-9.S, U1A.A5
- net N$28: now also BUS-38.S, U2A.A6; no longer BUS-10.S, U1A.A6
- net N$32: now also BUS-39.S, U2A.A7; no longer BUS-11.S, U1A.A7
- net N$33: now also BUS-40.S, U2A.A8; no longer BUS-12.S, U1A.A8
- net N$36: now also BUS-23.S, U1A.A1; no longer BUS-15.S, IC30A.A1
- net N$37: now also BUS-24.S, U1A.A2; no longer BUS-16.S, IC30A.A2
- net N$38: now also BUS-25.S, U1A.A3; no longer BUS-17.S, IC30A.A3
- net N$39: now also BUS-26.S, U1A.A4; no longer BUS-18.S, IC30A.A4
- net N$40: now also BUS-27.S, U1A.A5; no longer BUS-19.S, IC30A.A5
- net N$42: now also BUS-28.S, U1A.A6; no longer BUS-20.S, IC30A.A6
- net N$43: now also BUS-29.S, U1A.A7; no longer BUS-21.S, IC30A.A7
- net N$44: now also BUS-30.S, U1A.A8; no longer BUS-22.S, IC30A.A8
- net N$45: now also BUS-14.S, U3A.A1; no longer BUS-25.S, IC31A.A1
- net N$48: now also BUS-13.S, U3A.A2; no longer BUS-26.S, IC31A.A2
- net N$49: now also BUS-9.S, U3A.A3; no longer BUS-27.S, IC31A.A3
- net N$50: now also BUS-8.S, U3A.A4; no longer BUS-28.S, IC31A.A4
- net N$51: now also BUS-7.S, U3A.A5; no longer BUS-29.S, IC31A.A5
- net N$52: now also BUS-6.S, U3A.A7; no longer BUS-33.S, IC31A.A7
- net N$54: now also BUS-5.S, U3A.A8; no longer BUS-34.S, IC31A.A8
Other:
- moved on the sheet: SV4-23, SV4-24, SV4-25, SV4-26, SV4-27, SV4-28, SV4-29, SV4-30, SV4-31, SV4-32, SV4-33

Commit message: Finalise bus power pin assignments
Parts:
- removed C2: 220uF, rcl:CPOL-EUE3.5-8
Connections:
- net +5V: now also BUS-2.S, BUS-4.S, U9B.A, U9B.CLR; no longer BUS-1.S, BUS-3.S, C2.+
- net GND: now also BUS-1.S, BUS-3.S; no longer BUS-2.S, BUS-4.S, C2.-, U9B.A, U9B.CLR
- net N$19: now also BUS-23.S, U1A.A8; no longer BUS-33.S, U2A.A1
- net N$20: now also BUS-24.S, U1A.A7; no longer BUS-34.S, U2A.A2
- net N$22: now also BUS-25.S, U1A.A6; no longer BUS-35.S, U2A.A3
- net N$23: now also BUS-26.S, U1A.A5; no longer BUS-36.S, U2A.A4
- net N$26: now also BUS-27.S, U1A.A4; no longer BUS-37.S, U2A.A5
- net N$28: now also BUS-28.S, U1A.A3; no longer BUS-38.S, U2A.A6
- net N$32: now also BUS-29.S, U1A.A2; no longer BUS-39.S, U2A.A7
- net N$33: now also BUS-30.S, U1A.A1; no longer BUS-40.S, U2A.A8
- net N$36: now also BUS-33.S, U2A.A8; no longer BUS-23.S, U1A.A1
- net N$37: now also BUS-34.S, U2A.A7; no longer BUS-24.S, U1A.A2
- net N$38: now also BUS-35.S, U2A.A6; no longer BUS-25.S, U1A.A3
- net N$39: now also BUS-36.S, U2A.A5; no longer BUS-26.S, U1A.A4
- net N$40: now also BUS-37.S, U2A.A4; no longer BUS-27.S, U1A.A5
- net N$42: now also BUS-38.S, U2A.A3; no longer BUS-28.S, U1A.A6
- net N$43: now also BUS-39.S, U2A.A2; no longer BUS-29.S, U1A.A7
- net N$44: now also BUS-40.S, U2A.A1; no longer BUS-30.S, U1A.A8
Other:
- note added: "LAYOUT OF SHIFT REGISTERS AND RELATION TO HEADERS AS SEEN FROM BOTTOM OF DISPLAY DRIVER BOARD"
- note added: "SV1"
- note added: "SV2"
- note added: "SV3"
- note added: "SV4"
- note added: "U15"
- note added: "U16"
- note added: "U17"
- note added: "U18"
- note added: "U19"
- note added: "U20"
- note added: "U21"
- note added: "U22"
- note added: "U23"
- note added: "U24"
- note added: "U25"
- note added: "U26"
- note added: "U27"
- note added: "U28"
- note added: "U29"
- note added: "U30"
- note added: "U31"
- moved on the sheet: BUS-1, BUS-2, BUS-23, BUS-24, BUS-25, BUS-26, BUS-27, BUS-28, BUS-29, BUS-3, BUS-30, BUS-33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

Commit message: Reverse order of column shift regs
Connections:
- removed net COL5_B: R57.1, U21A.QH
- removed net COL7_F: R18.1, U17A.QA
- new net COL5\_B: R105.1, U27A.QH
- new net COL7\_F: R130.1, U31A.QA
- net COL0_A: now also R10.1, U16A.QA; no longer R122.1, U30A.QA
- net COL0_B: now also R25.1, U17A.QH; no longer R137.1, U31A.QH
- net COL0_C: now also R23.1, U17A.QF; no longer R135.1, U31A.QF
- net COL0_D: now also R20.1, U17A.QC; no longer R132.1, U31A.QC
- net COL0_E: now also R19.1, U17A.QB; no longer R131.1, U31A.QB
- net COL0_F: now also R18.1, U17A.QA; no longer R130.1, U31A.QA
- net COL0_G: now also R17.1, U16A.QH; no longer R129.1, U30A.QH
- net COL0_H: now also R13.1, U16A.QD; no longer R125.1, U30A.QD
- net COL0_K: now also R12.1, U16A.QC; no longer R124.1, U30A.QC
- net COL0_M: now also R11.1, U16A.QB; no longer R123.1, U30A.QB
- net COL0_N: now also R24.1, U17A.QG; no longer R136.1, U31A.QG
- net COL0_P: now also R22.1, U17A.QE; no longer R134.1, U31A.QE
- net COL0_R: now also R21.1, U17A.QD; no longer R133.1, U31A.QD
- net COL0_S: now also R15.1, U16A.QF; no longer R127.1, U30A.QF
- net COL0_T: now also R16.1, U16A.QG; no longer R128.1, U30A.QG
- net COL0_U: now also R14.1, U16A.QE; no longer R126.1, U30A.QE
- net COL1_A: now also R26.1, U18A.QA; no longer R106.1, U28A.QA
- net COL1_B: now also R41.1, U19A.QH; no longer R121.1, U29A.QH
- net COL1_C: now also R39.1, U19A.QF; no longer R119.1, U29A.QF
- net COL1_D: now also R36.1, U19A.QC; no longer R116.1, U29A.QC
- net COL1_E: now also R35.1, U19A.QB; no longer R115.1, U29A.QB
- net COL1_F: now also R34.1, U19A.QA; no longer R114.1, U29A.QA
- net COL1_G: now also R33.1, U18A.QH; no longer R113.1, U28A.QH
- net COL1_H: now also R29.1, U18A.QD; no longer R109.1, U28A.QD
- net COL1_K: now also R28.1, U18A.QC; no longer R108.1, U28A.QC
- net COL1_M: now also R27.1, U18A.QB; no longer R107.1, U28A.QB
- net COL1_N: now also R40.1, U19A.QG; no longer R120.1, U29A.QG
- net COL1_P: now also R38.1, U19A.QE; no longer R118.1, U29A.QE
- net COL1_R: now also R37.1, U19A.QD; no longer R117.1, U29A.QD
- net COL1_S: now also R31.1, U18A.QF; no longer R111.1, U28A.QF
- net COL1_T: now also R32.1, U18A.QG; no longer R112.1, U28A.QG
- net COL1_U: now also R30.1, U18A.QE; no longer R110.1, U28A.QE
- net COL2_A: now also R42.1, U20A.QA; no longer R90.1, U26A.QA
- net COL2_B: now also R57.1, U21A.QH; no longer R105.1, U27A.QH
- net COL2_C: now also R55.1, U21A.QF; no longer R103.1, U27A.QF
- net COL2_D: now also R52.1, U21A.QC; no longer R100.1, U27A.QC
- net COL2_E: now also R51.1, U21A.QB; no longer R99.1, U27A.QB
- net COL2_F: now also R50.1, U21A.QA; no longer R98.1, U27A.QA
- net COL2_G: now also R49.1, U20A.QH; no longer R97.1, U26A.QH
- net COL2_H: now also R45.1, U20A.QD; no longer R93.1, U26A.QD
- net COL2_K: now also R44.1, U20A.QC; no longer R92.1, U26A.QC
- net COL2_M: now also R43.1, U20A.QB; no longer R91.1, U26A.QB
- net COL2_N: now also R56.1, U21A.QG; no longer R104.1, U27A.QG
- net COL2_P: now also R54.1, U21A.QE; no longer R102.1, U27A.QE
- net COL2_R: now also R53.1, U21A.QD; no longer R101.1, U27A.QD
- net COL2_S: now also R47.1, U20A.QF; no longer R95.1, U26A.QF
- net COL2_T: now also R48.1, U20A.QG; no longer R96.1, U26A.QG
- net COL2_U: now also R46.1, U20A.QE; no longer R94.1, U26A.QE
- net COL3_A: now also R58.1, U22A.QA; no longer R74.1, U24A.QA
- net COL3_B: now also R73.1, U23A.QH; no longer R89.1, U25A.QH
- net COL3_C: now also R71.1, U23A.QF; no longer R87.1, U25A.QF
- net COL3_D: now also R68.1, U23A.QC; no longer R84.1, U25A.QC
- net COL3_E: now also R67.1, U23A.QB; no longer R83.1, U25A.QB
- net COL3_F: now also R66.1, U23A.QA; no longer R82.1, U25A.QA
- net COL3_G: now also R65.1, U22A.QH; no longer R81.1, U24A.QH
- net COL3_H: now also R61.1, U22A.QD; no longer R77.1, U24A.QD
- net COL3_K: now also R60.1, U22A.QC; no longer R76.1, U24A.QC
- net COL3_M: now also R59.1, U22A.QB; no longer R75.1, U24A.QB
- net COL3_N: now also R72.1, U23A.QG; no longer R88.1, U25A.QG
- net COL3_P: now also R70.1, U23A.QE; no longer R86.1, U25A.QE
- net COL3_R: now also R69.1, U23A.QD; no longer R85.1, U25A.QD
- net COL3_S: now also R63.1, U22A.QF; no longer R79.1, U24A.QF
- net COL3_T: now also R64.1, U22A.QG; no longer R80.1, U24A.QG
- net COL3_U: now also R62.1, U22A.QE; no longer R78.1, U24A.QE
- net COL4_A: now also R74.1, U24A.QA; no longer R58.1, U22A.QA
- net COL4_B: now also R89.1, U25A.QH; no longer R73.1, U23A.QH
- net COL4_C: now also R87.1, U25A.QF; no longer R71.1, U23A.QF
- net COL4_D: now also R84.1, U25A.QC; no longer R68.1, U23A.QC
- net COL4_E: now also R83.1, U25A.QB; no longer R67.1, U23A.QB
- net COL4_F: now also R82.1, U25A.QA; no longer R66.1, U23A.QA
- net COL4_G: now also R81.1, U24A.QH; no longer R65.1, U22A.QH
- net COL4_H: now also R77.1, U24A.QD; no longer R61.1, U22A.QD
- net COL4_K: now also R76.1, U24A.QC; no longer R60.1, U22A.QC
- net COL4_M: now also R75.1, U24A.QB; no longer R59.1, U22A.QB
- net COL4_N: now also R88.1, U25A.QG; no longer R72.1, U23A.QG
- net COL4_P: now also R86.1, U25A.QE; no longer R70.1, U23A.QE
- net COL4_R: now also R85.1, U25A.QD; no longer R69.1, U23A.QD
- net COL4_S: now also R79.1, U24A.QF; no longer R63.1, U22A.QF
- net COL4_T: now also R80.1, U24A.QG; no longer R64.1, U22A.QG
- net COL4_U: now also R78.1, U24A.QE; no longer R62.1, U22A.QE
- net COL5_A: now also R90.1, U26A.QA; no longer R42.1, U20A.QA
- net COL5_C: now also R103.1, U27A.QF; no longer R55.1, U21A.QF
- net COL5_D: now also R100.1, U27A.QC; no longer R52.1, U21A.QC
- net COL5_E: now also R99.1, U27A.QB; no longer R51.1, U21A.QB
- net COL5_F: now also R98.1, U27A.QA; no longer R50.1, U21A.QA
- net COL5_G: now also R97.1, U26A.QH; no longer R49.1, U20A.QH
- net COL5_H: now also R93.1, U26A.QD; no longer R45.1, U20A.QD
- net COL5_K: now also R92.1, U26A.QC; no longer R44.1, U20A.QC
- net COL5_M: now also R91.1, U26A.QB; no longer R43.1, U20A.QB
- net COL5_N: now also R104.1, U27A.QG; no longer R56.1, U21A.QG
- net COL5_P: now also R102.1, U27A.QE; no longer R54.1, U21A.QE
- net COL5_R: now also R101.1, U27A.QD; no longer R53.1, U21A.QD
- net COL5_S: now also R95.1, U26A.QF; no longer R47.1, U20A.QF
- net COL5_T: now also R96.1, U26A.QG; no longer R48.1, U20A.QG
- net COL5_U: now also R94.1, U26A.QE; no longer R46.1, U20A.QE
- net COL6_A: now also R106.1, U28A.QA; no longer R26.1, U18A.QA
- net COL6_B: now also R121.1, U29A.QH; no longer R41.1, U19A.QH
- net COL6_C: now also R119.1, U29A.QF; no longer R39.1, U19A.QF
- net COL6_D: now also R116.1, U29A.QC; no longer R36.1, U19A.QC
- net COL6_E: now also R115.1, U29A.QB; no longer R35.1, U19A.QB
- net COL6_F: now also R114.1, U29A.QA; no longer R34.1, U19A.QA
- net COL6_G: now also R113.1, U28A.QH; no longer R33.1, U18A.QH
- net COL6_H: now also R109.1, U28A.QD; no longer R29.1, U18A.QD
- net COL6_K: now also R108.1, U28A.QC; no longer R28.1, U18A.QC
- net COL6_M: now also R107.1, U28A.QB; no longer R27.1, U18A.QB
- net COL6_N: now also R120.1, U29A.QG; no longer R40.1, U19A.QG
- net COL6_P: now also R118.1, U29A.QE; no longer R38.1, U19A.QE
- net COL6_R: now also R117.1, U29A.QD; no longer R37.1, U19A.QD
- net COL6_S: now also R111.1, U28A.QF; no longer R31.1, U18A.QF
- net COL6_T: now also R112.1, U28A.QG; no longer R32.1, U18A.QG
- net COL6_U: now also R110.1, U28A.QE; no longer R30.1, U18A.QE
- net COL7_A: now also R122.1, U30A.QA; no longer R10.1, U16A.QA
- net COL7_B: now also R137.1, U31A.QH; no longer R25.1, U17A.QH
- net COL7_C: now also R135.1, U31A.QF; no longer R23.1, U17A.QF
- net COL7_D: now also R132.1, U31A.QC; no longer R20.1, U17A.QC
- net COL7_E: now also R131.1, U31A.QB; no longer R19.1, U17A.QB
- net COL7_G: now also R129.1, U30A.QH; no longer R17.1, U16A.QH
- net COL7_H: now also R125.1, U30A.QD; no longer R13.1, U16A.QD
- net COL7_K: now also R124.1, U30A.QC; no longer R12.1, U16A.QC
- net COL7_M: now also R123.1, U30A.QB; no longer R11.1, U16A.QB
- net COL7_N: now also R136.1, U31A.QG; no longer R24.1, U17A.QG
- net COL7_P: now also R134.1, U31A.QE; no longer R22.1, U17A.QE
- net COL7_R: now also R133.1, U31A.QD; no longer R21.1, U17A.QD
- net COL7_S: now also R127.1, U30A.QF; no longer R15.1, U16A.QF
- net COL7_T: now also R128.1, U30A.QG; no longer R16.1, U16A.QG
- net COL7_U: now also R126.1, U30A.QE; no longer R14.1, U16A.QE
Other:
- moved on the sheet: SV4-34, SV4-35, SV4-36
