File: display driver shift reg.sch (EAGLE design)
At the start: 205 parts, among them U1 74LS245N, U10 74HC32, U11 74HC166, U12 74HC08, U13 74HC573, U14 74HC138, U15 74HC595, U16 74HC595, U17 74HC595, U18 74HC595, U19 74HC595, U2 74LS245N, U20 74HC595, U21 74HC595, U22 74HC595, U23 74HC595, U24 74HC595, U25 74HC595, U26 74HC595, U27 74HC595, U28 74HC595, U29 74HC595, U3 74LS245N, U30 74HC595, U31 74HC595, U4 74HC688, U5 74HC688, U6 74HC04, U7 74HC74, U8 74HC08, U9 74HC393

Commit message: Re-assigned header pins to match new shift reg layout
Connections:
- net N$100: now also SV1-25.S; no longer SV2-1.S
- net N$101: now also SV1-26.S; no longer SV2-2.S
- net N$102: now also SV1-27.S; no longer SV2-3.S
- net N$103: now also SV1-28.S; no longer SV2-4.S
- net N$104: now also SV1-29.S; no longer SV2-5.S
- net N$105: now also SV1-30.S; no longer SV2-6.S
- net N$106: now also SV1-31.S; no longer SV2-7.S
- net N$107: now also SV1-32.S; no longer SV2-8.S
- net N$108: now also SV2-1.S; no longer SV2-33.S
- net N$109: now also SV2-2.S; no longer SV2-34.S
- net N$110: now also SV2-3.S; no longer SV2-35.S
- net N$111: now also SV2-4.S; no longer SV2-36.S
- net N$112: now also SV2-5.S; no longer SV2-37.S
- net N$113: now also SV2-6.S; no longer SV2-38.S
- net N$114: now also SV2-7.S; no longer SV2-39.S
- net N$115: now also SV2-8.S; no longer SV2-40.S
- net N$116: now also R58.2; no longer R106.2
- net N$117: now also R59.2; no longer R107.2
- net N$118: now also R60.2; no longer R108.2
- net N$119: now also R61.2; no longer R109.2
- net N$120: now also R62.2; no longer R110.2
- net N$121: now also R63.2; no longer R111.2
- net N$122: now also R64.2; no longer R112.2
- net N$123: now also R65.2; no longer R113.2
- net N$124: now also SV1-33.S; no longer SV2-9.S
- net N$125: now also SV1-34.S; no longer SV2-10.S
- net N$126: now also SV1-35.S; no longer SV2-11.S
- net N$127: now also SV1-36.S; no longer SV2-12.S
- net N$128: now also SV1-37.S; no longer SV2-13.S
- net N$129: now also SV1-38.S; no longer SV2-14.S
- net N$130: now also SV1-39.S; no longer SV2-15.S
- net N$131: now also SV1-40.S; no longer SV2-16.S
- net N$132: now also R66.2, SV3-33.S; no longer R82.2, SV3-1.S
- net N$133: now also R67.2, SV3-34.S; no longer R83.2, SV3-2.S
- net N$134: now also R68.2, SV3-35.S; no longer R84.2, SV3-3.S
- net N$135: now also R69.2, SV3-36.S; no longer R85.2, SV3-4.S
- net N$136: now also R70.2, SV3-37.S; no longer R86.2, SV3-5.S
- net N$137: now also R71.2, SV3-38.S; no longer R87.2, SV3-6.S
- net N$138: now also R72.2, SV3-39.S; no longer R88.2, SV3-7.S
- net N$139: now also R73.2, SV3-40.S; no longer R89.2, SV3-8.S
- net N$140: now also R82.2, SV2-9.S; no longer R114.2, SV3-33.S
- net N$141: now also R83.2, SV2-10.S; no longer R115.2, SV3-34.S
- net N$142: now also R84.2, SV2-11.S; no longer R116.2, SV3-35.S
- net N$143: now also R85.2, SV2-12.S; no longer R117.2, SV3-36.S
- net N$144: now also R86.2, SV2-13.S; no longer R118.2, SV3-37.S
- net N$145: now also R87.2, SV2-14.S; no longer R119.2, SV3-38.S
- net N$146: now also R88.2, SV2-15.S; no longer R120.2, SV3-39.S
- net N$147: now also R89.2, SV2-16.S; no longer R121.2, SV3-40.S
- net N$148: now also R90.2, SV4-1.S; no longer R58.2, SV2-17.S
- net N$149: now also R91.2, SV4-2.S; no longer R59.2, SV2-18.S
- net N$150: now also R92.2, SV4-3.S; no longer R60.2, SV2-19.S
- net N$151: now also R93.2, SV4-4.S; no longer R61.2, SV2-20.S
- net N$152: now also R94.2, SV4-5.S; no longer R62.2, SV2-21.S
- net N$153: now also R95.2, SV4-6.S; no longer R63.2, SV2-22.S
- net N$154: now also R96.2, SV4-7.S; no longer R64.2, SV2-23.S
- net N$155: now also R97.2, SV4-8.S; no longer R65.2, SV2-24.S
- net N$156: now also R98.2, SV4-9.S; no longer R90.2, SV3-9.S
- net N$157: now also R99.2, SV4-10.S; no longer R91.2, SV3-10.S
- net N$158: now also R100.2, SV4-11.S; no longer R92.2, SV3-11.S
- net N$159: now also R101.2, SV4-12.S; no longer R93.2, SV3-12.S
- net N$160: now also R102.2, SV4-13.S; no longer R94.2, SV3-13.S
- net N$161: now also R103.2, SV4-14.S; no longer R95.2, SV3-14.S
- net N$162: now also R104.2, SV4-15.S; no longer R96.2, SV3-15.S
- net N$163: now also R105.2, SV4-16.S; no longer R97.2, SV3-16.S
- net N$164: now also R106.2, SV2-17.S; no longer R122.2, SV4-1.S
- net N$165: now also R107.2, SV2-18.S; no longer R123.2, SV4-2.S
- net N$166: now also R108.2, SV2-19.S; no longer R124.2, SV4-3.S
- net N$167: now also R109.2, SV2-20.S; no longer R125.2, SV4-4.S
- net N$168: now also R110.2, SV2-21.S; no longer R126.2, SV4-5.S
- net N$169: now also R111.2, SV2-22.S; no longer R127.2, SV4-6.S
- net N$170: now also R112.2, SV2-23.S; no longer R128.2, SV4-7.S
- net N$171: now also R113.2, SV2-24.S; no longer R129.2, SV4-8.S
- net N$172: now also R114.2; no longer R66.2
- net N$173: now also R115.2; no longer R67.2
- net N$174: now also R116.2; no longer R68.2
- net N$175: now also R117.2; no longer R69.2
- net N$176: now also R118.2; no longer R70.2
- net N$177: now also R119.2; no longer R71.2
- net N$178: now also R120.2; no longer R72.2
- net N$179: now also R121.2; no longer R73.2
- net N$180: now also R122.2, SV2-33.S; no longer R98.2, SV3-17.S
- net N$181: now also R123.2, SV2-34.S; no longer R99.2, SV3-18.S
- net N$182: now also R124.2, SV2-35.S; no longer R100.2, SV3-19.S
- net N$183: now also R125.2, SV2-36.S; no longer R101.2, SV3-20.S
- net N$184: now also R126.2, SV2-37.S; no longer R102.2, SV3-21.S
- net N$185: now also R127.2, SV2-38.S; no longer R103.2, SV3-22.S
- net N$186: now also R128.2, SV2-39.S; no longer R104.2, SV3-23.S
- net N$187: now also R129.2, SV2-40.S; no longer R105.2, SV3-24.S
- net N$188: now also SV4-17.S; no longer SV4-9.S
- net N$189: now also SV4-18.S; no longer SV4-10.S
- net N$190: now also SV4-19.S; no longer SV4-11.S
- net N$191: now also SV4-20.S; no longer SV4-12.S
- net N$192: now also SV4-21.S; no longer SV4-13.S
- net N$193: now also SV4-22.S; no longer SV4-14.S
- net N$194: now also SV4-23.S; no longer SV4-15.S
- net N$195: now also SV4-24.S; no longer SV4-16.S
- net N$84: now also SV3-1.S; no longer SV1-25.S
- net N$85: now also SV3-2.S; no longer SV1-26.S
- net N$86: now also SV3-3.S; no longer SV1-27.S
- net N$87: now also SV3-4.S; no longer SV1-28.S
- net N$88: now also SV3-5.S; no longer SV1-29.S
- net N$89: now also SV3-6.S; no longer SV1-30.S
- net N$90: now also SV3-7.S; no longer SV1-31.S
- net N$91: now also SV3-8.S; no longer SV1-32.S
- net N$92: now also SV3-9.S; no longer SV1-33.S
- net N$93: now also SV3-10.S; no longer SV1-34.S
- net N$94: now also SV3-11.S; no longer SV1-35.S
- net N$95: now also SV3-12.S; no longer SV1-36.S
- net N$96: now also SV3-13.S; no longer SV1-37.S
- net N$97: now also SV3-14.S; no longer SV1-38.S
- net N$98: now also SV3-15.S; no longer SV1-39.S
- net N$99: now also SV3-16.S; no longer SV1-40.S
Other:
- moved on the sheet: SV1-25, SV1-26, SV1-27, SV1-28, SV1-29, SV1-30, SV1-31, SV1-32, SV1-33, SV1-34, SV1-35, SV1-36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
