File: schematics/16 seg display board.sch (EAGLE design)
At the start: 14 parts, among them Q1 BC327, Q2 BC327, Q3 BC327

Commit message: First attempt at board layout
Parts:
- removed LED2, LED3, LED4, LED5, LED6, LED7, LED8: PSA08-11SYKWA, Z80 clock:PSA08-11SYKWA
- added CN1, CN2, CN3, CN4: (no value), Z80 clock:HDR40
- added LED_R1C1, LED_R1C2, LED_R1C3, LED_R1C4, LED_R1C5, LED_R1C6, LED_R1C7, LED_R2C0, LED_R2C1, LED_R2C2, LED_R2C3, LED_R2C4, LED_R2C5, LED_R2C6, LED_R2C7, LED_R3C0, LED_R3C1, LED_R3C2, LED_R3C3, LED_R3C4, LED_R3C5, LED_R3C6, LED_R3C7: PSA08-11SYKWA, Z80 clock:PSA08-11SYKWA
- Q1, Q2, Q3: value BC327 -> BD438; device transistor-pnp:BC327 -> transistor-power:BD438
- renumbered LED1 to LED_R1C0
Connections:
- new net COL0_A: CN1-16.S, LED_R1C0.A, LED_R2C0.A, LED_R3C0.A
- new net COL0_B: CN1-17.S, LED_R1C0.B, LED_R2C0.B, LED_R3C0.B
- new net COL0_C: CN1-19.S, LED_R1C0.C, LED_R2C0.C, LED_R3C0.C
- new net COL0_D: CN1-22.S, LED_R1C0.D, LED_R2C0.D, LED_R3C0.D
- new net COL0_E: CN1-23.S, LED_R1C0.E, LED_R2C0.E, LED_R3C0.E
- new net COL0_F: CN1-24.S, LED_R1C0.F, LED_R2C0.F, LED_R3C0.F
- new net COL0_G: CN1-9.S, LED_R1C0.G, LED_R2C0.G, LED_R3C0.G
- new net COL0_H: CN1-13.S, LED_R1C0.H, LED_R2C0.H, LED_R3C0.H
- new net COL0_K: CN1-14.S, LED_R1C0.K, LED_R2C0.K, LED_R3C0.K
- new net COL0_M: CN1-15.S, LED_R1C0.M, LED_R2C0.M, LED_R3C0.M
- new net COL0_N: CN1-18.S, LED_R1C0.N, LED_R2C0.N, LED_R3C0.N
- new net COL0_P: CN1-20.S, LED_R1C0.P, LED_R2C0.P, LED_R3C0.P
- new net COL0_R: CN1-21.S, LED_R1C0.R, LED_R2C0.R, LED_R3C0.R
- new net COL0_S: CN1-11.S, LED_R1C0.S, LED_R2C0.S, LED_R3C0.S
- new net COL0_T: CN1-10.S, LED_R1C0.T, LED_R2C0.T, LED_R3C0.T
- new net COL0_U: CN1-12.S, LED_R1C0.U, LED_R2C0.U, LED_R3C0.U
- new net COL1_A: CN3-5.S, LED_R1C1.A, LED_R2C1.A, LED_R3C1.A
- new net COL1_B: CN3-12.S, LED_R1C1.B, LED_R2C1.B, LED_R3C1.B
- new net COL1_C: CN3-10.S, LED_R1C1.C, LED_R2C1.C, LED_R3C1.C
- new net COL1_D: CN3-15.S, LED_R1C1.D, LED_R2C1.D, LED_R3C1.D
- new net COL1_E: CN3-14.S, LED_R1C1.E, LED_R2C1.E, LED_R3C1.E
- new net COL1_F: CN3-13.S, LED_R1C1.F, LED_R2C1.F, LED_R3C1.F
- new net COL1_G: CN3-4.S, LED_R1C1.G, LED_R2C1.G, LED_R3C1.G
- new net COL1_H: CN3-8.S, LED_R1C1.H, LED_R2C1.H, LED_R3C1.H
- new net COL1_K: CN3-7.S, LED_R1C1.K, LED_R2C1.K, LED_R3C1.K
- new net COL1_M: CN3-6.S, LED_R1C1.M, LED_R2C1.M, LED_R3C1.M
- new net COL1_N: CN3-11.S, LED_R1C1.N, LED_R2C1.N, LED_R3C1.N
- new net COL1_P: CN3-9.S, LED_R1C1.P, LED_R2C1.P, LED_R3C1.P
- new net COL1_R: CN3-16.S, LED_R1C1.R, LED_R2C1.R, LED_R3C1.R
- new net COL1_S: CN3-2.S, LED_R1C1.S, LED_R2C1.S, LED_R3C1.S
- new net COL1_T: CN3-3.S, LED_R1C1.T, LED_R2C1.T, LED_R3C1.T
- new net COL1_U: CN3-1.S, LED_R1C1.U, LED_R2C1.U, LED_R3C1.U
- new net COL2_A: CN1-32.S, LED_R1C2.A, LED_R2C2.A, LED_R3C2.A
- new net COL2_B: CN1-33.S, LED_R1C2.B, LED_R2C2.B, LED_R3C2.B
- new net COL2_C: CN1-35.S, LED_R1C2.C, LED_R2C2.C, LED_R3C2.C
- new net COL2_D: CN1-38.S, LED_R1C2.D, LED_R2C2.D, LED_R3C2.D
- new net COL2_E: CN1-39.S, LED_R1C2.E, LED_R2C2.E, LED_R3C2.E
- new net COL2_F: CN1-40.S, LED_R1C2.F, LED_R2C2.F, LED_R3C2.F
- new net COL2_G: CN1-25.S, LED_R1C2.G, LED_R2C2.G, LED_R3C2.G
- new net COL2_H: CN1-29.S, LED_R1C2.H, LED_R2C2.H, LED_R3C2.H
- new net COL2_K: CN1-30.S, LED_R1C2.K, LED_R2C2.K, LED_R3C2.K
- new net COL2_M: CN1-31.S, LED_R1C2.M, LED_R2C2.M, LED_R3C2.M
- new net COL2_N: CN1-34.S, LED_R1C2.N, LED_R2C2.N, LED_R3C2.N
- new net COL2_P: CN1-36.S, LED_R1C2.P, LED_R2C2.P, LED_R3C2.P
- new net COL2_R: CN1-37.S, LED_R1C2.R, LED_R2C2.R, LED_R3C2.R
- new net COL2_S: CN1-27.S, LED_R1C2.S, LED_R2C2.S, LED_R3C2.S
- new net COL2_T: CN1-26.S, LED_R1C2.T, LED_R2C2.T, LED_R3C2.T
- new net COL2_U: CN1-28.S, LED_R1C2.U, LED_R2C2.U, LED_R3C2.U
- new net COL3_A: CN3-29.S, LED_R1C3.A, LED_R2C3.A, LED_R3C3.A
- new net COL3_B: CN3-36.S, LED_R1C3.B, LED_R2C3.B, LED_R3C3.B
- new net COL3_C: CN3-34.S, LED_R1C3.C, LED_R2C3.C, LED_R3C3.C
- new net COL3_D: CN3-39.S, LED_R1C3.D, LED_R2C3.D, LED_R3C3.D
- new net COL3_E: CN3-38.S, LED_R1C3.E, LED_R2C3.E, LED_R3C3.E
- new net COL3_F: CN3-37.S, LED_R1C3.F, LED_R2C3.F, LED_R3C3.F
- new net COL3_G: CN3-28.S, LED_R1C3.G, LED_R2C3.G, LED_R3C3.G
- new net COL3_H: CN3-32.S, LED_R1C3.H, LED_R2C3.H, LED_R3C3.H
- new net COL3_K: CN3-31.S, LED_R1C3.K, LED_R2C3.K, LED_R3C3.K
- new net COL3_M: CN3-30.S, LED_R1C3.M, LED_R2C3.M, LED_R3C3.M
- new net COL3_N: CN3-35.S, LED_R1C3.N, LED_R2C3.N, LED_R3C3.N
- new net COL3_P: CN3-33.S, LED_R1C3.P, LED_R2C3.P, LED_R3C3.P
- new net COL3_R: CN3-40.S, LED_R1C3.R, LED_R2C3.R, LED_R3C3.R
- new net COL3_S: CN3-26.S, LED_R1C3.S, LED_R2C3.S, LED_R3C3.S
- new net COL3_T: CN3-27.S, LED_R1C3.T, LED_R2C3.T, LED_R3C3.T
- new net COL3_U: CN3-25.S, LED_R1C3.U, LED_R2C3.U, LED_R3C3.U
- new net COL4\_C: CN2-11.S, LED_R1C4.C, LED_R2C4.C, LED_R3C4.C
- new net COL4_A: CN2-8.S, LED_R1C4.A, LED_R2C4.A, LED_R3C4.A
- new net COL4_B: CN2-9.S, LED_R1C4.B, LED_R2C4.B, LED_R3C4.B
- new net COL4_D: CN2-14.S, LED_R1C4.D, LED_R2C4.D, LED_R3C4.D
- new net COL4_E: CN2-15.S, LED_R1C4.E, LED_R2C4.E, LED_R3C4.E
- new net COL4_F: CN2-16.S, LED_R1C4.F, LED_R2C4.F, LED_R3C4.F
- new net COL4_G: CN2-1.S, LED_R1C4.G, LED_R2C4.G, LED_R3C4.G
- new net COL4_H: CN2-5.S, LED_R1C4.H, LED_R2C4.H, LED_R3C4.H
- new net COL4_K: CN2-6.S, LED_R1C4.K, LED_R2C4.K, LED_R3C4.K
- new net COL4_M: CN2-7.S, LED_R1C4.M, LED_R2C4.M, LED_R3C4.M
- new net COL4_N: CN2-10.S, LED_R1C4.N, LED_R2C4.N, LED_R3C4.N
- new net COL4_P: CN2-12.S, LED_R1C4.P, LED_R2C4.P, LED_R3C4.P
- new net COL4_R: CN2-13.S, LED_R1C4.R, LED_R2C4.R, LED_R3C4.R
- new net COL4_S: CN2-3.S, LED_R1C4.S, LED_R2C4.S, LED_R3C4.S
- new net COL4_T: CN2-2.S, LED_R1C4.T, LED_R2C4.T, LED_R3C4.T
- new net COL4_U: CN2-4.S, LED_R1C4.U, LED_R2C4.U, LED_R3C4.U
- new net COL5\_S: CN4-2.S, LED_R1C5.S, LED_R2C5.S, LED_R3C5.S
- new net COL5\_U: CN4-1.S, LED_R1C5.U, LED_R2C5.U, LED_R3C5.U
- new net COL5_A: CN4-5.S, LED_R1C5.A, LED_R2C5.A, LED_R3C5.A
- new net COL5_B: CN4-12.S, LED_R1C5.B, LED_R2C5.B, LED_R3C5.B
- new net COL5_C: CN4-10.S, LED_R1C5.C, LED_R2C5.C, LED_R3C5.C
- new net COL5_D: CN4-15.S, LED_R1C5.D, LED_R2C5.D, LED_R3C5.D
- new net COL5_E: CN4-14.S, LED_R1C5.E, LED_R2C5.E, LED_R3C5.E
- new net COL5_F: CN4-13.S, LED_R1C5.F, LED_R2C5.F, LED_R3C5.F
- new net COL5_G: CN4-4.S, LED_R1C5.G, LED_R2C5.G, LED_R3C5.G
- new net COL5_H: CN4-8.S, LED_R1C5.H, LED_R2C5.H, LED_R3C5.H
- new net COL5_K: CN4-7.S, LED_R1C5.K, LED_R2C5.K, LED_R3C5.K
- new net COL5_M: CN4-6.S, LED_R1C5.M, LED_R2C5.M, LED_R3C5.M
- new net COL5_N: CN4-11.S, LED_R1C5.N, LED_R2C5.N, LED_R3C5.N
- new net COL5_P: CN4-9.S, LED_R1C5.P, LED_R2C5.P, LED_R3C5.P
- new net COL5_R: CN4-16.S, LED_R1C5.R, LED_R2C5.R, LED_R3C5.R
- new net COL5_T: CN4-3.S, LED_R1C5.T, LED_R2C5.T, LED_R3C5.T
- new net COL6_A: CN2-24.S, LED_R1C6.A, LED_R2C6.A, LED_R3C6.A
- new net COL6_B: CN2-25.S, LED_R1C6.B, LED_R2C6.B, LED_R3C6.B
- new net COL6_C: CN2-27.S, LED_R1C6.C, LED_R2C6.C, LED_R3C6.C
- new net COL6_D: CN2-30.S, LED_R1C6.D, LED_R2C6.D, LED_R3C6.D
- new net COL6_E: CN2-31.S, LED_R1C6.E, LED_R2C6.E, LED_R3C6.E
- new net COL6_F: CN2-32.S, LED_R1C6.F, LED_R2C6.F, LED_R3C6.F
- new net COL6_G: CN2-17.S, LED_R1C6.G, LED_R2C6.G, LED_R3C6.G
- new net COL6_H: CN2-21.S, LED_R1C6.H, LED_R2C6.H, LED_R3C6.H
- new net COL6_K: CN2-22.S, LED_R1C6.K, LED_R2C6.K, LED_R3C6.K
- new net COL6_M: CN2-23.S, LED_R1C6.M, LED_R2C6.M, LED_R3C6.M
- new net COL6_N: CN2-26.S, LED_R1C6.N, LED_R2C6.N, LED_R3C6.N
- new net COL6_P: CN2-28.S, LED_R1C6.P, LED_R2C6.P, LED_R3C6.P
- new net COL6_R: CN2-29.S, LED_R1C6.R, LED_R2C6.R, LED_R3C6.R
- new net COL6_S: CN2-19.S, LED_R1C6.S, LED_R2C6.S, LED_R3C6.S
- new net COL6_T: CN2-18.S, LED_R1C6.T, LED_R2C6.T, LED_R3C6.T
- new net COL6_U: CN2-20.S, LED_R1C6.U, LED_R2C6.U, LED_R3C6.U
- new net COL7_A: CN2-40.S, LED_R1C7.A, LED_R2C7.A, LED_R3C7.A
- new net COL7_B: CN4-20.S, LED_R1C7.B, LED_R2C7.B, LED_R3C7.B
- new net COL7_C: CN4-18.S, LED_R1C7.C, LED_R2C7.C, LED_R3C7.C
- new net COL7_D: CN4-23.S, LED_R1C7.D, LED_R2C7.D, LED_R3C7.D
- new net COL7_E: CN4-22.S, LED_R1C7.E, LED_R2C7.E, LED_R3C7.E
- new net COL7_F: CN4-21.S, LED_R1C7.F, LED_R2C7.F, LED_R3C7.F
- new net COL7_G: CN2-33.S, LED_R1C7.G, LED_R2C7.G, LED_R3C7.G
- new net COL7_H: CN2-37.S, LED_R1C7.H, LED_R2C7.H, LED_R3C7.H
- new net COL7_K: CN2-38.S, LED_R1C7.K, LED_R2C7.K, LED_R3C7.K
- new net COL7_M: CN2-39.S, LED_R1C7.M, LED_R2C7.M, LED_R3C7.M
- new net COL7_N: CN4-19.S, LED_R1C7.N, LED_R2C7.N, LED_R3C7.N
- new net COL7_P: CN4-17.S, LED_R1C7.P, LED_R2C7.P, LED_R3C7.P
- new net COL7_R: CN4-24.S, LED_R1C7.R, LED_R2C7.R, LED_R3C7.R
- new net COL7_S: CN2-35.S, LED_R1C7.S, LED_R2C7.S, LED_R3C7.S
- new net COL7_T: CN2-34.S, LED_R1C7.T, LED_R2C7.T, LED_R3C7.T
- new net COL7_U: CN2-36.S, LED_R1C7.U, LED_R2C7.U, LED_R3C7.U
- new net DP0: CN1-8.S, LED_R1C0.DP, LED_R2C0.DP, LED_R3C0.DP
- new net DP1: CN1-7.S, LED_R1C1.DP, LED_R2C1.DP, LED_R3C1.DP
- new net DP2: CN1-6.S, LED_R1C2.DP, LED_R2C2.DP, LED_R3C2.DP
- new net DP3: CN1-5.S, LED_R1C3.DP, LED_R2C3.DP, LED_R3C3.DP
- new net DP4: CN1-4.S, LED_R1C4.DP, LED_R2C4.DP, LED_R3C4.DP
- new net DP5: CN1-3.S, LED_R1C5.DP, LED_R2C5.DP, LED_R3C5.DP
- new net DP6: CN1-2.S, LED_R1C6.DP, LED_R2C6.DP, LED_R3C6.DP
- new net DP7: CN1-1.S, LED_R1C7.DP, LED_R2C7.DP, LED_R3C7.DP
- new net GND: CN4-37.S, CN4-39.S
- new net N$4: CN4-34.S, R1.1
- new net N$5: CN4-35.S, R2.1
- new net N$6: CN4-36.S, R3.1
- new net R1_PWR: LED_R1C0.CA, LED_R1C1.CA, LED_R1C2.CA, LED_R1C3.CA, LED_R1C4.CA, LED_R1C5.CA, LED_R1C6.CA, LED_R1C7.CA, Q1.C
- new net R2_PWR: LED_R2C0.CA, LED_R2C1.CA, LED_R2C2.CA, LED_R2C3.CA, LED_R2C4.CA, LED_R2C5.CA, LED_R2C6.CA, LED_R2C7.CA, Q2.C
- new net R3_PWR: LED_R3C0.CA, LED_R3C1.CA, LED_R3C2.CA, LED_R3C3.CA, LED_R3C4.CA, LED_R3C5.CA, LED_R3C6.CA, LED_R3C7.CA, Q3.C
- net +5V: now also CN4-38.S, CN4-40.S
