File: schematics/timer rtc io.sch (EAGLE design)
At the start: 78 parts, among them T1 BC547, U1 74HC245, U10 74HC688, U11 74HC30, U12 74HC00, U13 74HC32, U14 74HC04, U15 74HC08, U16 74HC688, U17 74HC138, U18 74HC138, U19 74HC573, U2 74HC245, U20 74HC573, U21 74HC573, U22 74HC573, U23 74HC573, U24 NE555, U3 74HC245, U4 74HC688, U6 74HC74, U7 74HC590, U8 74HC688, U9 BQ4845, X1 32.768KHz, Y1 4.096MHz

Commit message: First attempt at board layout
Parts:
- removed C25: 100nF, rcl:C-EU050-025X075
- removed U18: 74HC138, 74xx-us:74LS138N
- added JP3: (no value), jumper:JP2E
- added JP4: (no value), Z80 clock:JP3Q
- BUS: device con-ml:ML40E -> Z80 clock:HDR40
- JP1: device jumper:JP3Q -> Z80 clock:JP3Q
- U5: value (none) -> Z84C30
Connections:
- removed net N$52 (its old number): U13D.O, U18A.G2B
- removed net N$64: RN2-1.1, U5.TRG0
- new net CTC_CH2: JP3.3, U5.TO2
- new net N$61: JP3.1, U24.OUT
- new net N$62: JP3.2, R2.1
- new net N$92: JP4.6, RN2-3.1, U5.TRG2
- net !IORQ!: no longer U13B.I0, U13C.I0
- net !M1!: now also U13D.I1; no longer U13C.I1
- net !RD!: no longer U13B.I1
- net !RESET!: now also U12D.I0; no longer U12D.I1
- net !WR!: no longer U13D.I1
- net +5V: now also U10A.Q1, U16A.Q6, U8A.Q2; no longer C25.1, U10A.Q2, U16A.Q3, U18A.G1, U18P.VCC, U8A.Q4
- net A0: no longer U18A.A
- net A1: now also U10A.P7; no longer U10A.P1, U18A.B
- net A2: now also U10A.P1, U4A.P1; no longer U10A.P2, U18A.C, U4A.P2
- net A3: now also U10A.P6, U16A.P6, U4A.P6; no longer U10A.P3, U16A.P3, U4A.P3
- net A4: now also U10A.P2, U16A.P2, U4A.P2, U8A.P2; no longer U10A.P4, U16A.P4, U4A.P4, U8A.P4
- net A6: now also U10A.P3, U16A.P3, U4A.P3, U8A.P3; no longer U10A.P6, U16A.P6, U4A.P6, U8A.P6
- net A7: now also U10A.P4, U16A.P4, U4A.P4, U8A.P4; no longer U10A.P7, U16A.P7, U4A.P7, U8A.P7
- net GND: now also SW1.S, SW1.S1, SW2.S, SW2.S1, SW3.S, SW3.S1, SW4.S, SW4.S1, U10A.Q2, U13B.I0, U13B.I1, U13C.I0, U13C.I1, U16A.P7, U16A.Q3, U17A.G2B, U4A.P7, U8A.P6, U8A.P7, U8A.Q4; no longer C25.2, SW1.P, SW1.P1, SW2.P, SW2.P1, SW3.P, SW3.P1, SW4.P, SW4.P1, U10A.Q1, U16A.P2, U16A.Q6, U18P.GND, U4A.P1, U8A.P2, U8A.P3, U8A.Q2
- net N$10: no longer U18A.G2A
- net N$11: now also JP4.4, RN2-2.1, U5.TRG1; no longer U13B.O, U17A.G2B
- net N$3: now also U11A.I0; no longer U11A.I1
- net N$37: now also SW1.P1; no longer SW1.S, SW1.S1
- net N$38: now also SW2.P1; no longer SW2.S, SW2.S1
- net N$39: now also SW3.P; no longer SW3.S, SW3.S1
- net N$40: now also SW4.P1; no longer SW4.S, SW4.S1
- net N$45: now also U11A.I2; no longer U11A.I3
- net N$46: now also U11A.I3; no longer U11A.I4
- net N$47: now also U11A.I6; no longer U11A.I5
- net N$48: now also U15A.I0; no longer U15A.I1
- net N$5: now also U11A.I4; no longer U11A.I0
- net N$50: now also JP4.2, RN2-1.1, U5.TRG0; no longer RN2-3.1, U5.TRG2
- net N$54: now also U12D.I1, U17A.Y4; no longer U12D.I0, U18A.Y4
- net N$59: now also JP4.1, JP4.3, JP4.5; no longer RN2-2.1, U5.TRG1
- net N$60: now also T1.C; no longer U24.OUT
- net N$7: now also U11A.I1; no longer U11A.I2
- net N$87: now also U15A.I1; no longer U15A.I0
- net N$90: now also U11A.I5; no longer U11A.I6
- net N$91: now also U13D.O; no longer U13C.O
Other:
- note added: "CH0 DISPLAY REFRESH CH1 10MS MAIN LOOP CH2 SPEAKER CH3 RTC"
- note removed: "TODO"
- moved on the sheet: BAT1, BUS-15, C26, C27, C28, JP2, R1, R2, R4, R5, RN2-1, RN2-2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

Commit message: Finalise PCB layout for timer/rtc/io board
Moved the CTC and RTC chips to the unbuffed side of the data bus, and modified direction and enable logic for data bus buffer
Parts:
- removed C14, C15, C16: 100nF, rcl:C-EU050-025X075
- removed U13: 74HC32, 74xx-us:74LS32N
- removed U14: 74HC04, 74xx-us:74LS04N
- removed U15: 74HC08, 74xx-us:74LS08N
- BAT1: device battery:CR2032H -> Z80 clock:CR2032-SMD
- SG1: value F/CM12P -> PKM13EPYH4000X; device buzzer:F/CM12P -> Z80 clock:PKM13EPYH4000X
Connections:
- removed net DIR: U15A.O, U1A.DIR
- removed net N$48: U13A.O, U15A.I0
- removed net N$49: BUS-23.S, U1A.A8
- removed net N$51: U12A.I1, U14F.O
- removed net N$65: BUS-24.S, U1A.A7
- removed net N$66: BUS-25.S, U1A.A6
- removed net N$67: BUS-26.S, U1A.A5
- removed net N$68: BUS-27.S, U1A.A4
- removed net N$69: BUS-28.S, U1A.A3
- removed net N$70: BUS-29.S, U1A.A2
- removed net N$71: BUS-30.S, U1A.A1
- removed net N$87: U12A.O, U15A.I1
- removed net N$91: U13A.I1, U13D.O
- new net !OBD!: U12C.O, U1A.G
- new net D0`: BUS-30.S, U1A.A1, U5.D0, U9.D0
- new net D1`: BUS-29.S, U1A.A2, U5.D1, U9.D1
- new net D2`: BUS-28.S, U1A.A3, U5.D2, U9.D2
- new net D3`: BUS-27.S, U1A.A4, U5.D3, U9.D3
- new net D4`: BUS-26.S, U1A.A5, U5.D4, U9.D4
- new net D5`: BUS-25.S, U1A.A6, U5.D5, U9.D5
- new net D6`: BUS-24.S, U1A.A7, U5.D6, U9.D6
- new net D7`: BUS-23.S, U1A.A8, U5.D7, U9.D7
- new net N$64: U4A.P=Q, U5.CE
- net !IEO!: no longer U13A.I0
- net !IORQ!: no longer U13D.I0
- net !M1!: no longer U13D.I1
- net !RD!: now also U1A.DIR; no longer U14F.I
- net !RESET!: no longer U14A.I
- net +5V: now also U11A.I3, U11A.I4, U11A.I5, U12C.I1; no longer C14.1, C15.1, C16.1, U13P.VCC, U14P.VCC, U15P.VCC
- net D0: no longer U5.D0, U9.D0
- net D1: no longer U5.D1, U9.D1
- net D2: no longer U5.D2, U9.D2
- net D3: no longer U5.D3, U9.D3
- net D4: no longer U5.D4, U9.D4
- net D5: no longer U5.D5, U9.D5
- net D6: no longer U5.D6, U9.D6
- net D7: no longer U5.D7, U9.D7
- net GND: now also U12A.I0, U12A.I1; no longer C14.2, C15.2, C16.2, U12C.I0, U12C.I1, U13B.I0, U13B.I1, U13C.I0, U13C.I1, U13P.GND, U14B.I, U14C.I, U14D.I, U14E.I, U14P.GND, U15B.I0, U15B.I1, U15C.I0, U15C.I1, U15D.I0, U15D.I1, U15P.GND
- net N$1: no longer JP1.3
- net N$3: no longer U11A.I0
- net N$36: now also JP1.5, U6B.Q; no longer U11A.O, U12A.I0
- net N$45: now also U11A.I0; no longer U11A.I2
- net N$46: now also U11A.I1; no longer U11A.I3
- net N$5: now also U11A.O, U12C.I0; no longer U11A.I4, U8A.P=Q, U9.!CS!
- net N$58: no longer JP1.5
- net N$7: now also U8A.P=Q, U9.!CS!; no longer U11A.I1, U4A.P=Q, U5.CE
- net N$9: now also JP1.3, U6A.Q; no longer U14A.O, U1A.G
- net N$90: now also U11A.I2; no longer U11A.I5
Other:
- moved on the sheet: BUS-23, BUS-24, BUS-25, BUS-26, BUS-27, BUS-28, BUS-29, BUS-30, C17, C18, C19, C20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
